File: imu.kicad_sch (KiCad schematic)
At the start: 2 parts, among them U5 LSM6DSOTR

Commit message: Update footprints and add JLCPCB fields
Update some footprints which will suit better building the pcb
with JLCBPCB. Add fields to components sourced from JLCPCB
to be able to generate BOM.
Parts:
- C18: JLC (none) -> 0402; LCSC (none) -> C1525
- U5: JLC (none) -> LGA-14(2.5x3); LCSC (none) -> C2655100
Changed lines of the file:
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@@
+      (effects (font (size 1.27 1.27)) hide)
+    )
+    (property "JLC" "LGA-14(2.5x3)" (id 4) (at 151.13 94.615 0)
+      (effects (font (size 1.27 1.27)) hide)
+    )
+    (property "LCSC" "C2655100" (id 5) (at 151.13 94.615 0)
       (effects (font (size 1.27 1.27)) hide)
     )
@@
       (effects (font (size 1.27 1.27)) hide)
     )
+    (property "JLC" "0402" (id 4) (at 160.655 72.39 0)
+      (effects (font (size 1.27 1.27)) hide)
+    )
+    (property "LCSC" "C1525" (id 5) (at 160.655 72.39 0)
+      (effects (font (size 1.27 1.27)) hide)
+    )
